File: board/board.kicad_sch (KiCad schematic)
At the start: 1 part

Commit message: imported legacy version
Parts:
- added J1: 004_BASE-T_CT_2x3, on_edge:on_edge_2x05_device, symbol put_on_edge:004_BASE-T_CT
- added J2: 013_PoE_rectified, on_edge:on_edge_2x05_host, symbol put_on_edge:013_PoE_rectified
- LOGO1: footprint Symbol:OSHW-Symbol_6.7x6mm_SilkScreen -> Symbol:OSHW-Logo2_9.8x8mm_SilkScreen
Connections:
- new net GND: J1.1 (GND), J1.10 (GND), J1.3 (GND), J1.5 (GND), J1.7 (GND), J1.9 (GND), J2.1 (GND), J2.2 (GND), J2.5 (GND)
- new net snippet/CT1: J1.2 (CT1)
- new net snippet/CT2: J1.4 (CT2)
- new net snippet/CT3: J1.6 (CT3)
- new net snippet/CT4: J1.8 (CT4)
- new net snippet/P: J2.3 (48V), J2.4 (48V)
Other:
- removed sheet implementation
- added sheet snippet (snippet.kicad_sch)
- note removed: "Input connectors go here"
- note removed: "Output connectors go here"
